File: sch/ESP32-TestPatternGenerator/ESP32-TestPatternGenerator.kicad_sch (KiCad schematic)
At the start: 4 parts, among them J1 Composite Video Out, SW1 Format, SW2 Pattern

Commit message: first pass of the PCB
Parts:
- SW1, SW2: footprint (none) -> Button_Switch_THT:SW_PUSH_6mm_H4.3mm
Changed lines of the file:
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@@
       (effects (font (size 1.27 1.27)))
     )
-    (property "Footprint" "" (at 107.95 87.63 0)
+    (property "Footprint" "Button_Switch_THT:SW_PUSH_6mm_H4.3mm" (at 107.95 87.63 0)
       (effects (font (size 1.27 1.27)) hide)
     )
@@
       (effects (font (size 1.27 1.27)))
     )
-    (property "Footprint" "" (at 107.95 74.93 0)
+    (property "Footprint" "Button_Switch_THT:SW_PUSH_6mm_H4.3mm" (at 107.95 74.93 0)
       (effects (font (size 1.27 1.27)) hide)
     )

Commit message: minor changes
Parts:
- J1: footprint (none) -> RCJ-044:CUI_RCJ-044
- LOLIND32: footprint (none) -> Wemos:LOLIN_D32
Changed lines of the file:
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@@
       (effects (font (size 1.27 1.27)) (justify left))
     )
-    (property "Footprint" "" (at 119.38 67.31 0)
+    (property "Footprint" "RCJ-044:CUI_RCJ-044" (at 119.38 67.31 0)
       (effects (font (size 1.27 1.27)) hide)
     )
@@
       (effects (font (size 1.27 1.27)))
     )
-    (property "Footprint" "" (at 96.52 74.93 0)
+    (property "Footprint" "Wemos:LOLIN_D32" (at 96.52 74.93 0)
       (effects (font (size 1.27 1.27)) hide)
     )
